File: hw/dummy_load/load.kicad_sch (KiCad schematic)
At the start: 33 parts, among them Q2 IRL540NPBF, Q3 IRL540NPBF, Q4 IRL540NPBF, Q5 IRL540NPBF, Q6 IRL540NPBF, Q7 IRL540NPBF, Q8 IRL540NPBF, Q9 IRL540NPBF

Commit message: Replace terminal block, update BOM and datasheets, minor fixes to tracing
Signed-off-by: Mateusz Pajak <22417805+Tai-Min@users.noreply.github.com>
Parts:
- HS1: LCSC Part # (none) -> https://www.tme.com/us/en-us/details/sk68-50sa/heatsinks/fi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
Changed lines of the file:
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@@
 			)
 		)
-		(property "LCSC Part #" "~"
+		(property "LCSC Part #" "https://www.tme.com/us/en-us/details/sk68-50sa/heatsinks/fischer-elektronik/"
 			(at 232.41 74.93 0)
 			(effects

Commit message: Better PCB design, update BOM, add UART header for debugging (#7)
Signed-off-by: Mateusz Pajak <22417805+Tai-Min@users.noreply.github.com>
Parts:
- R42, R43, R44, R45, R46, R47, R48, R49: footprint Resistor_SMD:R_1206_3216Metric_Pad1.30x1.75mm_HandSolder -> Resistor_SMD:R_0603_1608Metric; LCSC Part # C706405 -> C22548
- R50, R52, R54, R56, R58, R60, R62, R64: footprint Resistor_SMD:R_1206_3216Metric_Pad1.30x1.75mm_HandSolder -> Resistor_SMD:R_0603_1608Metric; LCSC Part # C2907517 -> C2907181
- R51, R53, R55, R57, R59, R61, R63, R65: footprint Resistor_SMD:R_2512_6332Metric_Pad1.40x3.35mm_HandSolder -> Resistor_SMD:R_2512_6332Metric
Changed lines of the file:
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@@
 			)
 		)
-		(property "Footprint" "Resistor_SMD:R_1206_3216Metric_Pad1.30x1.75mm_HandSolder"
+		(property "Footprint" "Resistor_SMD:R_0603_1608Metric"
 			(at 103.378 87.63 90)
 			(effects
@@
 			)
 		)
-		(property "LCSC Part #" "C2907517"
+		(property "LCSC Part #" "C2907181"
 			(at 101.6 87.63 0)
 			(effects
@@
 			)
 		)
-		(property "Footprint" "Resistor_SMD:R_2512_6332Metric_Pad1.40x3.35mm_HandSolder"
+		(property "Footprint" "Resistor_SMD:R_2512_6332Metric"
 			(at 149.352 113.03 90)
 			(effects
@@
 			)
 		)
-		(property "Footprint" "Resistor_SMD:R_2512_6332Metric_Pad1.40x3.35mm_HandSolder"
+		(property "Footprint" "Resistor_SMD:R_2512_6332Metric"
 			(at 230.632 113.03 90)
 			(effects
@@
 			)
 		)
-		(property "Footprint" "Resistor_SMD:R_2512_6332Metric_Pad1.40x3.35mm_HandSolder"
+		(property "Footprint" "Resistor_SMD:R_2512_6332Metric"
 			(at 129.032 113.03 90)
 			(effects
@@
 			)
 		)
-		(property "Footprint" "Resistor_SMD:R_2512_6332Metric_Pad1.40x3.35mm_HandSolder"
+		(property "Footprint" "Resistor_SMD:R_2512_6332Metric"
 			(at 210.312 113.03 90)
 			(effects
@@
 			)
 		)
-		(property "Footprint" "Resistor_SMD:R_1206_3216Metric_Pad1.30x1.75mm_HandSolder"
+		(property "Footprint" "Resistor_SMD:R_0603_1608Metric"
 			(at 71.12 122.682 90)
 			(effects
@@
 			)
 		)
-		(property "LCSC Part #" "C706405"
+		(property "LCSC Part #" "C22548"
 			(at 71.12 124.46 90)
 			(effects
@@
 			)
 		)
-		(property "Footprint" "Resistor_SMD:R_2512_6332Metric_Pad1.40x3.35mm_HandSolder"
+		(property "Footprint" "Resistor_SMD:R_2512_6332Metric"
 			(at 169.672 113.03 90)
 			(effects
@@
 			)
 		)
-		(property "Footprint" "Resistor_SMD:R_1206_3216Metric_Pad1.30x1.75mm_HandSolder"
+		(property "Footprint" "Resistor_SMD:R_0603_1608Metric"
 			(at 204.978 87.63 90)
 			(effects
@@
 			)
 		)
-		(property "LCSC Part #" "C2907517"
+		(property "LCSC Part #" "C2907181"
 			(at 203.2 87.63 0)
 			(effects
@@
 			)
 		)
-		(property "Footprint" "Resistor_SMD:R_1206_3216Metric_Pad1.30x1.75mm_HandSolder"
+		(property "Footprint" "Resistor_SMD:R_0603_1608Metric"
 			(at 184.658 87.63 90)
 			(effects
@@
 			)
 		)
-		(property "LCSC Part #" "C2907517"
+		(property "LCSC Part #" "C2907181"
 			(at 182.88 87.63 0)
 			(effects
@@
 			)
 		)
-		(property "Footprint" "Resistor_SMD:R_1206_3216Metric_Pad1.30x1.75mm_HandSolder"
+		(property "Footprint" "Resistor_SMD:R_0603_1608Metric"
 			(at 164.338 87.63 90)
 			(effects
@@
 			)
 		)
-		(property "LCSC Part #" "C2907517"
+		(property "LCSC Part #" "C2907181"
 			(at 162.56 87.63 0)
 			(effects
@@
 			)
 		)
-		(property "Footprint" "Resistor_SMD:R_1206_3216Metric_Pad1.30x1.75mm_HandSolder"
+		(property "Footprint" "Resistor_SMD:R_0603_1608Metric"
 			(at 71.12 135.382 90)
 			(effects
@@
 			)
 		)
-		(property "LCSC Part #" "C706405"
+		(property "LCSC Part #" "C22548"
 			(at 71.12 137.16 90)
 			(effects
@@
 			)
 		)
-		(property "Footprint" "Resistor_SMD:R_1206_3216Metric_Pad1.30x1.75mm_HandSolder"
+		(property "Footprint" "Resistor_SMD:R_0603_1608Metric"
 			(at 83.058 87.63 90)
 			(effects
@@
 			)
 		)
-		(property "LCSC Part #" "C2907517"
+		(property "LCSC Part #" "C2907181"
 			(at 81.28 87.63 0)
 			(effects
@@
 			)
 		)
-		(property "Footprint" "Resistor_SMD:R_1206_3216Metric_Pad1.30x1.75mm_HandSolder"
+		(property "Footprint" "Resistor_SMD:R_0603_1608Metric"
 			(at 71.12 109.982 90)
 			(effects
@@
 			)
 		)
-		(property "LCSC Part #" "C706405"
+		(property "LCSC Part #" "C22548"
 			(at 71.12 111.76 90)
 			(effects
@@
 			)
 		)
-		(property "Footprint" "Resistor_SMD:R_1206_3216Metric_Pad1.30x1.75mm_HandSolder"
+		(property "Footprint" "Resistor_SMD:R_0603_1608Metric"
 			(at 144.018 87.63 90)
 			(effects
@@
 			)
 		)
-		(property "LCSC Part #" "C2907517"
+		(property "LCSC Part #" "C2907181"
 			(at 142.24 87.63 0)
 			(effects
@@
 			)
 		)
-		(property "Footprint" "Resistor_SMD:R_1206_3216Metric_Pad1.30x1.75mm_HandSolder"
+		(property "Footprint" "Resistor_SMD:R_0603_1608Metric"
 			(at 71.12 129.032 90)
 			(effects
@@
 			)
 		)
-		(property "LCSC Part #" "C706405"
+		(property "LCSC Part #" "C22548"
 			(at 71.12 130.81 90)
 			(effects
@@
 			)
 		)
-		(property "Footprint" "Resistor_SMD:R_1206_3216Metric_Pad1.30x1.75mm_HandSolder"
+		(property "Footprint" "Resistor_SMD:R_0603_1608Metric"
 			(at 123.698 87.63 90)
 			(effects
@@
 			)
 		)
-		(property "LCSC Part #" "C2907517"
+		(property "LCSC Part #" "C2907181"
 			(at 121.92 87.63 0)
 			(effects
@@
 			)
 		)
-		(property "Footprint" "Resistor_SMD:R_1206_3216Metric_Pad1.30x1.75mm_HandSolder"
+		(property "Footprint" "Resistor_SMD:R_0603_1608Metric"
 			(at 71.12 116.332 90)
 			(effects
@@
 			)
 		)
-		(property "LCSC Part #" "C706405"
+		(property "LCSC Part #" "C22548"
 			(at 71.12 118.11 90)
 			(effects
@@
 			)
 		)
-		(property "Footprint" "Resistor_SMD:R_1206_3216Metric_Pad1.30x1.75mm_HandSolder"
+		(property "Footprint" "Resistor_SMD:R_0603_1608Metric"
 			(at 71.12 103.632 90)
 			(effects
@@
 			)
 		)
-		(property "LCSC Part #" "C706405"
+		(property "LCSC Part #" "C22548"
 			(at 71.12 105.41 90)
 			(effects
@@
 			)
 		)
-		(property "Footprint" "Resistor_SMD:R_2512_6332Metric_Pad1.40x3.35mm_HandSolder"
+		(property "Footprint" "Resistor_SMD:R_2512_6332Metric"
 			(at 108.712 113.03 90)
 			(effects
@@
 			)
 		)
-		(property "Footprint" "Resistor_SMD:R_2512_6332Metric_Pad1.40x3.35mm_HandSolder"
+		(property "Footprint" "Resistor_SMD:R_2512_6332Metric"
 			(at 189.992 113.03 90)
 			(effects
@@
 			)
 		)
-		(property "Footprint" "Resistor_SMD:R_2512_6332Metric_Pad1.40x3.35mm_HandSolder"
+		(property "Footprint" "Resistor_SMD:R_2512_6332Metric"
 			(at 88.392 113.03 90)
 			(effects
@@
 			)
 		)
-		(property "Footprint" "Resistor_SMD:R_1206_3216Metric_Pad1.30x1.75mm_HandSolder"
+		(property "Footprint" "Resistor_SMD:R_0603_1608Metric"
 			(at 71.12 141.732 90)
 			(effects
@@
 			)
 		)
-		(property "LCSC Part #" "C706405"
+		(property "LCSC Part #" "C22548"
 			(at 71.12 143.51 90)
 			(effects
@@
 			)
 		)
-		(property "Footprint" "Resistor_SMD:R_1206_3216Metric_Pad1.30x1.75mm_HandSolder"
+		(property "Footprint" "Resistor_SMD:R_0603_1608Metric"
 			(at 225.298 87.63 90)
 			(effects
@@
 			)
 		)
-		(property "LCSC Part #" "C2907517"
+		(property "LCSC Part #" "C2907181"
 			(at 223.52 87.63 0)
 			(effects
@@
 			)
 		)
-		(property "Footprint" "Resistor_SMD:R_1206_3216Metric_Pad1.30x1.75mm_HandSolder"
+		(property "Footprint" "Resistor_SMD:R_0603_1608Metric"
 			(at 71.12 97.282 90)
 			(effects
@@
 			)
 		)
-		(property "LCSC Part #" "C706405"
+		(property "LCSC Part #" "C22548"
 			(at 71.12 99.06 90)
 			(effects
